File: Jetson_camera_interposer.kicad_pcb (KiCad board)
At the start: 6 copper layers, 82.1 x 75 mm, 20 parts, among them J1 QSH-060-01-L-D-A, J2 QTH-060-01-L-D-A, J21 Conn_01x01, J22 Conn_01x01, J23 Conn_01x01, J24 Conn_01x01, J25 Conn_01x01, J26 Conn_01x01, J3 Conn_01x01, J4 Conn_01x01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

Commit message: organized footprints
Parts:
- added J9: Conn_02x30_Odd_Even, Pin_Headers:Pin_Header_Straight_2x06_Pitch2.54mm, F.Cu at (94.0, 134.6)
- moved J8 56.3 mm to (161.3, 72.2)
Connections:
- J7 pad 1: /VDD_SYS_J -> /VDD_SYS
- J7 pad 2: /VDD_SYS -> /VDD_SYS_J
- J7 pad 3: /VDD_IR_J -> /VDD_IR
- J7 pad 4: /VDD_IR -> /VDD_IR_J
- J8 pad 10: (no net) -> /CAM0_RST
- J8 pad 12: (no net) -> /CAM0_MCLK
- J8 pad 14: (no net) -> /I2C_GP0_DAT_1V8
- J8 pad 16: (no net) -> /I2C_GP0_CLK_1V8
- J8 pad 18: (no net) -> /CAM_I2C2_SDA
- J8 pad 2: (no net) -> /CAM2_RST
- J8 pad 20: (no net) -> /CAM_I2C2_SCL
- J8 pad 22: (no net) -> /I2C_CAM_DAT
- J8 pad 24: (no net) -> /I2C_CAM_CLK
- J8 pad 4: (no net) -> /CAM2_MCLK
- J8 pad 6: (no net) -> /CAM1_RST_L
- J8 pad 8: (no net) -> /CAM1_MCLK
Routing:
- net /VDD_IR_J: track 73.7 -> 65.4 mm, vias 1 -> 2
- net /VDD_SYS_J: track 60.6 -> 56.5 mm
- net /VDD_SYS: track 40.7 -> 43.7 mm, vias 1 -> 2
- net /VDD_AF: track 30.0 -> 27.7 mm
- net /AVDD_CAM: track 41.0 -> 38.7 mm
- net /VDD_IR: track 35.2 -> 36.9 mm
- net /VDD_3V3: track 36.1 -> 35.0 mm
- net /JETSON_1V8: track 31.0 -> 30.0 mm
- net /VDD_3V3_J: track 56.6 -> 55.7 mm
- net /VDD_AF_J: track 52.4 -> 51.6 mm
- net /AVDD_CAM_J: track 54.9 -> 54.3 mm
- net Earth: vias 245 -> 247

Commit message: finished routing second connector
Connections:
- I2C_CLK2 pad 1: /I2C_GP0_CLK_1V8 -> /I2C_GP0_CLK_1V8_J
- I2C_DAT2 pad 1: /I2C_GP0_DAT_1V8 -> /I2C_GP0_DAT_1V8_J
- J1 pad 105: /I2C_GP0_CLK_1V8 -> /I2C_GP0_CLK_1V8_J
- J1 pad 107: /I2C_GP0_DAT_1V8 -> /I2C_GP0_DAT_1V8_J
- J1 pad 75: /I2C_CAM_CLK -> /I2C_CAM_CLK_J
- J1 pad 77: /I2C_CAM_DAT -> /I2C_CAM_DAT_J
- J1 pad 87: /CAM_I2C2_SCL -> /CAM_I2C2_SCL_J
- J1 pad 88: /CAM1_MCLK -> /CAM1_MCLK_J
- J1 pad 89: /CAM_I2C2_SDA -> /CAM_I2C2_SDA_J
- J1 pad 91: /CAM0_MCLK -> /CAM0_MCLK_J
- J1 pad 92: /CAM1_RST_L -> /CAM1_RST_L_J
- J1 pad 94: /CAM2_MCLK -> /CAM2_MCLK_J
- J1 pad 95: /CAM0_RST -> /CAM0_RST_J
- J1 pad 98: /CAM2_RST -> /CAM2_RST_J
- J2 pad 95: /CAM0_RST -> /CAM0_RST_J
- J8 pad 1: (no net) -> /CAM2_RST_J
- J8 pad 10: /CAM0_RST -> (no net)
- J8 pad 11: (no net) -> /CAM0_MCLK_J
- J8 pad 13: (no net) -> /I2C_GP0_DAT_1V8_J
- J8 pad 15: (no net) -> /I2C_GP0_CLK_1V8_J
- J8 pad 17: (no net) -> /CAM_I2C2_SDA_J
- J8 pad 19: (no net) -> /CAM_I2C2_SCL_J
- J8 pad 21: (no net) -> /I2C_CAM_DAT_J
- J8 pad 23: (no net) -> /I2C_CAM_CLK_J
- J8 pad 3: (no net) -> /CAM2_MCLK_J
- J8 pad 5: (no net) -> /CAM1_RST_L_J
- J8 pad 7: (no net) -> /CAM1_MCLK_J
- J8 pad 9: (no net) -> /CAM0_RST_J
Routing:
- net /CAM2_RST: track 0.00 -> 80.9 mm, vias 0 -> 1
- net /CAM2_MCLK: track 0.00 -> 79.8 mm
- net /I2C_GP0_DAT_1V8: track 0.00 -> 75.1 mm, vias 0 -> 1
- net /CAM1_MCLK: track 0.00 -> 71.5 mm
- net /CAM1_RST_L: track 0.00 -> 62.3 mm, vias 0 -> 1
- net /CAM2_MCLK_J: track 0.00 -> 53.9 mm
- net /CAM0_MCLK: track 0.00 -> 46.6 mm
- net /I2C_GP0_CLK_1V8: track 0.00 -> 45.7 mm, vias 0 -> 1
- net /I2C_CAM_CLK: track 0.00 -> 43.9 mm
- net /CAM_I2C2_SCL: track 0.00 -> 43.6 mm
- net /CAM_I2C2_SDA: track 0.00 -> 42.7 mm
- net /I2C_CAM_DAT: track 0.00 -> 42.7 mm
- net /CAM1_MCLK_J: track 0.00 -> 42.0 mm
- net /CAM0_RST_J: track 0.00 -> 40.3 mm, vias 0 -> 1
- net /CAM2_RST_J: track 0.00 -> 30.4 mm, vias 0 -> 1
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
Commit message: finished third connector
Connections:
- J1 pad 117: /CAM_INTR -> /CAM_INTR_J
- J1 pad 119: /VSYS_EN -> /VSYS_EN_J
- J1 pad 86: /CAM_VSYNC -> /CAM_VSYNC_J
- J1 pad 90: /CAM1_PWDN -> /CAM1_PWDN_J
- J1 pad 93: /CAM0_PWR -> /CAM0_PWR_J
- J1 pad 96: /CAM2_PWDN -> /CAM2_PWDN_J
- J9 pad 1: (no net) -> /CAM0_PWR_J
- J9 pad 10: (no net) -> /VSYS_EN
- J9 pad 11: (no net) -> /CAM_VSYNC_J
- J9 pad 12: (no net) -> /CAM_VSYNC
- J9 pad 2: (no net) -> /CAM0_PWR
- J9 pad 3: (no net) -> /CAM1_PWDN_J
- J9 pad 4: (no net) -> /CAM1_PWDN
- J9 pad 5: (no net) -> /CAM2_PWDN_J
- J9 pad 6: (no net) -> /CAM2_PWDN
- J9 pad 7: (no net) -> /CAM_INTR_J
- J9 pad 8: (no net) -> /CAM_INTR
- J9 pad 9: (no net) -> /VSYS_EN_J
Routing:
- net /CAM0_PWR_J: track 0.00 -> 102.2 mm, vias 0 -> 2
- net /CAM_INTR_J: track 0.00 -> 98.7 mm, vias 0 -> 3
- net /VSYS_EN_J: track 0.00 -> 95.7 mm, vias 0 -> 3
- net /CAM1_PWDN_J: track 0.00 -> 95.5 mm, vias 0 -> 3
- net /CAM2_PWDN_J: track 0.00 -> 84.3 mm, vias 0 -> 1
- net /CAM_INTR: track 0.00 -> 79.5 mm, vias 0 -> 2
- net /CAM_VSYNC_J: track 0.00 -> 67.4 mm, vias 0 -> 2
- net /CAM0_PWR: track 0.00 -> 66.7 mm, vias 0 -> 1
- net /CAM1_PWDN: track 0.00 -> 58.7 mm, vias 0 -> 1
- net /CAM2_PWDN: track 0.00 -> 56.9 mm, vias 0 -> 1
- net /CAM_VSYNC: track 0.00 -> 49.0 mm, vias 0 -> 2
- net /VSYS_EN: track 26.7 -> 71.9 mm, vias 2 -> 3
- net /AVDD_CAM_J: track 54.3 -> 51.1 mm
- net /CAM0_MCLK: track 46.6 -> 44.5 mm
- net /CAM1_RST_L: track 62.3 -> 63.0 mm

Commit message: clean up
Routing:
- net /VDD_CAM_FQ_HV_CAM: track 95.4 -> 59.9 mm, vias 1 -> 2
Changed lines of the file:
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@@
     (thickness 1.6)
     (drawings 14)
-    (tracks 2913)
+    (tracks 2910)
     (zones 0)
     (modules 21)
@@
   (via (at 127.26 122.06) (size 0.508) (drill 0.254) (layers F.Cu B.Cu) (net 1))
   (via (at 132.34 122.06) (size 0.508) (drill 0.254) (layers F.Cu B.Cu) (net 1))
-  (via (at 134.88 122.06) (size 0.508) (drill 0.254) (layers F.Cu B.Cu) (net 1))
+  (via (at 135.128 122.06) (size 0.508) (drill 0.254) (layers F.Cu B.Cu) (net 1))
   (via (at 137.42 122.06) (size 0.508) (drill 0.254) (layers F.Cu B.Cu) (net 1))
   (via (at 135.38 107.11) (size 0.508) (drill 0.254) (layers F.Cu B.Cu) (net 1))
@@
   (segment (start 96.928999 90.878999) (end 97.64 91.59) (width 0.254) (layer In3.Cu) (net 23))
   (segment (start 97.64 91.59) (end 97.64 91.61) (width 0.254) (layer In3.Cu) (net 23))
-  (segment (start 147.493552 94.77959) (end 146.946448 94.77959) (width 0.4064) (layer In3.Cu) (net 23))
-  (segment (start 147.88041 95.166448) (end 147.493552 94.77959) (width 0.4064) (layer In3.Cu) (net 23))
-  (segment (start 147.88041 95.713552) (end 147.88041 95.166448) (width 0.4064) (layer In3.Cu) (net 23))
-  (segment (start 97.64 91.61) (end 98.183012 92.153012) (width 0.4064) (layer In3.Cu) (net 23))
-  (segment (start 140.033552 103.56041) (end 147.88041 95.713552) (width 0.4064) (layer In3.Cu) (net 23))
-  (segment (start 104.76041 103.56041) (end 140.033552 103.56041) (width 0.4064) (layer In3.Cu) (net 23))
-  (segment (start 146.946448 94.77959) (end 143.936038 97.79) (width 0.4064) (layer In3.Cu) (net 23))
+  (segment (start 104.76041 103.56041) (end 129.36159 103.56041) (width 0.4064) (layer In3.Cu) (net 23))
   (segment (start 98.183012 96.983012) (end 104.76041 103.56041) (width 0.4064) (layer In3.Cu) (net 23))
+  (segment (start 97.64 91.61) (end 98.183012 92.153012) (width 0.4064) (layer In3.Cu) (net 23))
+  (segment (start 129.36159 103.56041) (end 130.302 102.62) (width 0.4064) (layer In3.Cu) (net 23))
   (segment (start 98.183012 92.153012) (end 98.183012 96.983012) (width 0.4064) (layer In3.Cu) (net 23))
-  (via (at 131.33 97.79) (size 0.3556) (drill 0.2032) (layers F.Cu B.Cu) (net 23))
-  (segment (start 143.936038 97.79) (end 131.33 97.79) (width 0.4064) (layer In3.Cu) (net 23))
-  (segment (start 131.078553 97.79) (end 131.33 97.79) (width 0.4064) (layer B.Cu) (net 23))
-  (segment (start 128.83 97.79) (end 131.078553 97.79) (width 0.4064) (layer B.Cu) (net 23))
-  (segment (start 126.54 95.5) (end 128.83 97.79) (width 0.4064) (layer B.Cu) (net 23))
-  (segment (start 124.47 95.5) (end 126.54 95.5) (width 0.4064) (layer B.Cu) (net 23))
+  (via (at 130.302 102.62) (size 0.3556) (drill 0.2032) (layers F.Cu B.Cu) (net 23))
+  (segment (start 130.302 102.62) (end 130.302 102.368553) (width 0.4064) (layer In2.Cu) (net 23))
+  (segment (start 130.124201 98.292201) (end 130.302 98.47) (width 0.4064) (layer B.Cu) (net 23))
+  (segment (start 127.332 95.5) (end 130.124201 98.292201) (width 0.4064) (layer B.Cu) (net 23))
+  (segment (start 130.302 102.368553) (end 130.302 98.47) (width 0.4064) (layer In2.Cu) (net 23))
+  (segment (start 124.47 95.5) (end 127.332 95.5) (width 0.4064) (layer B.Cu) (net 23))
+  (via (at 130.302 98.47) (size 0.3556) (drill 0.2032) (layers F.Cu B.Cu) (net 23))
   (via (at 118.84 97.87) (size 0.3556) (drill 0.2032) (layers F.Cu B.Cu) (net 24))
   (segment (start 117.832915 95.75046) (end 116.91136 95.75046) (width 0.254) (layer B.Cu) (net 24))
@@
   (segment (start 136.37776 94.75224) (end 135.9 95.23) (width 0.2032) (layer F.Cu) (net 93))
   (segment (start 143.34012 94.75224) (end 136.37776 94.75224) (width 0.2032) (layer F.Cu) (net 93))
-  (segment (start 135.9 95.23) (end 130.87 100.26) (width 0.2032) (layer In2.Cu) (net 93))
-  (segment (start 130.87 100.26) (end 130.87 123.53) (width 0.2032) (layer In2.Cu) (net 93))
   (via (at 126.99 127.63) (size 0.3556) (drill 0.2032) (layers F.Cu B.Cu) (net 93))
-  (segment (start 126.99 127.41) (end 126.99 127.63) (width 0.2032) (layer In2.Cu) (net 93))
-  (segment (start 130.87 123.53) (end 126.99 127.41) (width 0.2032) (layer In2.Cu) (net 93))
   (segment (start 126.99 127.63) (end 126.99 128.49) (width 0.2032) (layer In3.Cu) (net 93))
   (segment (start 126.99 128.49) (end 123.57 131.91) (width 0.2032) (layer In3.Cu) (net 93))
@@
   (segment (start 111.61 134.62) (end 106.68 134.62) (width 0.2032) (layer In3.Cu) (net 93))
   (segment (start 114.32 131.91) (end 111.61 134.62) (width 0.2032) (layer In3.Cu) (net 93))
+  (segment (start 126.99 127.41) (end 126.99 127.63) (width 0.2032) (layer In2.Cu) (net 93))
+  (segment (start 131.572 122.828) (end 126.99 127.41) (width 0.2032) (layer In2.Cu) (net 93))
+  (segment (start 131.572 99.558) (end 131.572 122.828) (width 0.2032) (layer In2.Cu) (net 93))
+  (segment (start 135.9 95.23) (end 131.572 99.558) (width 0.2032) (layer In2.Cu) (net 93))
   (via (at 140.51 96.51) (size 0.3556) (drill 0.2032) (layers F.Cu B.Cu) (net 94))
   (via (at 140.09 92.72) (size 0.3556) (drill 0.2032) (layers F.Cu B.Cu) (net 94))

Commit message: reset all wirings
Parts:
- removed J7: Conn_02x10_Odd_Even, Pin_Headers:Pin_Header_Straight_2x10_Pitch2.54mm
- removed J9: Conn_02x30_Odd_Even, Pin_Headers:Pin_Header_Straight_2x06_Pitch2.54mm
- moved J8 66.4 mm to (94.9, 70.8)
Connections:
- J1 pad 101: /JETSON_1V2_J -> /JETSON_1V2
- J1 pad 102: /JETSON_1V8_J -> /JETSON_1V8
- J1 pad 108: /VDD_3V3_J -> /VDD_3V3
- J1 pad 109: /VDD_IR_J -> /VDD_IR
- J1 pad 110: /VDD_3V3_J -> /VDD_3V3
- J1 pad 117: /CAM_INTR_J -> /CAM_INTR
- J1 pad 118: /VDD_SYS_J -> /VDD_SYS
- J1 pad 119: /VSYS_EN_J -> /VSYS_EN
- J1 pad 120: /VDD_SYS_J -> /VDD_SYS
- J1 pad 55: /DVDD_CAM_LV_J -> /DVDD_CAM_LV
- J1 pad 56: /DVDD_CAM_LV_J -> /DVDD_CAM_LV
- J1 pad 57: /DVDD_CAM_LV_J -> /DVDD_CAM_LV
- J1 pad 58: /DVDD_CAM_LV_J -> /DVDD_CAM_LV
- J1 pad 81: /VDD_CAM_FQ_HV_CAM_J -> /VDD_CAM_FQ_HV_CAM
- J1 pad 82: /AVDD_CAM_J -> /AVDD_CAM
- J1 pad 83: /VDD_CAM_FQ_HV_CAM_J -> /VDD_CAM_FQ_HV_CAM
- J1 pad 84: /VDD_AF_J -> /VDD_AF
- J1 pad 86: /CAM_VSYNC_J -> /CAM_VSYNC
- J1 pad 90: /CAM1_PWDN_J -> /CAM1_PWDN
- J1 pad 93: /CAM0_PWR_J -> /CAM0_PWR
- J1 pad 96: /CAM2_PWDN_J -> /CAM2_PWDN
Routing:
- net /CAM0_PWR_J: track 102.2 -> 0.00 mm, vias 2 -> 0
- net /CAM_INTR_J: track 98.7 -> 0.00 mm, vias 3 -> 0
- net /VSYS_EN_J: track 95.7 -> 0.00 mm, vias 3 -> 0
- net /CAM1_PWDN_J: track 95.5 -> 0.00 mm, vias 3 -> 0
- net /CAM2_PWDN_J: track 84.3 -> 0.00 mm, vias 1 -> 0
- net /CAM2_RST: track 80.9 -> 0.00 mm, vias 1 -> 0
- net /CAM2_MCLK: track 79.7 -> 0.00 mm
- net /CAM_INTR: track 79.5 -> 0.00 mm, vias 2 -> 0
- net /I2C_GP0_DAT_1V8: track 75.1 -> 0.00 mm, vias 1 -> 0
- net /VSYS_EN: track 71.9 -> 0.00 mm, vias 3 -> 0
- net /CAM1_MCLK: track 71.5 -> 0.00 mm
- net /CAM_VSYNC_J: track 67.4 -> 0.00 mm, vias 2 -> 0
- net /CAM0_PWR: track 66.7 -> 0.00 mm, vias 1 -> 0
- net /DVDD_CAM_LV_J: track 66.0 -> 0.00 mm, vias 1 -> 0
- net /VDD_CAM_FQ_HV_CAM_J: track 65.8 -> 0.00 mm, vias 1 -> 0
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
Commit message: leaving only single connector
Connections:
- J1 pad 117: /CAM_INTR -> (no net)
- J1 pad 119: /VSYS_EN -> (no net)
- J1 pad 55: /DVDD_CAM_LV -> /DVDD_CAM_LV_J
- J1 pad 57: /DVDD_CAM_LV -> /DVDD_CAM_LV_J
- J1 pad 86: /CAM_VSYNC -> (no net)
- J1 pad 90: /CAM1_PWDN -> (no net)
- J1 pad 93: /CAM0_PWR -> (no net)
- J1 pad 96: /CAM2_PWDN -> (no net)
- J2 pad 117: /CAM_INTR -> (no net)
- J2 pad 119: /VSYS_EN -> (no net)
- J2 pad 86: /CAM_VSYNC -> (no net)
- J2 pad 90: /CAM1_PWDN -> (no net)
- J2 pad 93: /CAM0_PWR -> (no net)
- J2 pad 96: /CAM2_PWDN -> (no net)
Routing:
- net /CAM0_MCLK_J: track 0.00 -> 31.6 mm
- net /CAM0_RST_J: track 0.00 -> 30.9 mm
- net /I2C_CAM_CLK_J: track 0.00 -> 29.5 mm
- net /I2C_GP0_DAT_1V8_J: track 0.00 -> 28.7 mm
- net /CAM0_MCLK: track 0.00 -> 28.1 mm
- net /I2C_GP0_CLK_1V8_J: track 0.00 -> 27.9 mm
- net /CAM_I2C2_SDA_J: track 0.00 -> 26.5 mm
- net /CAM_I2C2_SCL_J: track 0.00 -> 26.4 mm
- net /I2C_CAM_DAT_J: track 0.00 -> 25.7 mm
- net /I2C_GP0_DAT_1V8: track 0.00 -> 25.0 mm
- net /CAM_I2C2_SCL: track 0.00 -> 24.4 mm
- net /CAM_I2C2_SDA: track 0.00 -> 24.4 mm
- net /I2C_CAM_DAT: track 0.00 -> 24.2 mm
- net /I2C_CAM_CLK: track 0.00 -> 23.9 mm
- net /I2C_GP0_CLK_1V8: track 0.00 -> 23.7 mm
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
Commit message: continue routing
Connections:
- J1 pad 55: /DVDD_CAM_LV_J -> /DVDD_CAM_LV
- J1 pad 57: /DVDD_CAM_LV_J -> /DVDD_CAM_LV
- J1 pad 86: (no net) -> /CAM_VSYNC
- J2 pad 86: (no net) -> /CAM_VSYNC
- J2 pad 95: /CAM0_RST_J -> /CAM0_RST
- J8 pad 10: (no net) -> /CAM0_RST
Routing:
- net /CAM1_RST_L_J: track 0.00 -> 61.8 mm, vias 0 -> 1
- net /CAM2_RST_J: track 0.00 -> 57.1 mm
- net /CAM2_MCLK_J: track 0.00 -> 56.5 mm
- net /CAM1_MCLK_J: track 0.00 -> 55.0 mm
- net /CAM1_RST_L: track 0.00 -> 39.7 mm, vias 0 -> 1
- net /VDD_IR: track 0.00 -> 35.4 mm, vias 0 -> 1
- net /I2S3_SDOUT: track 0.00 -> 34.4 mm, vias 0 -> 3
- net /CAM_I2C2_SCL_J: track 26.4 -> 60.2 mm, vias 0 -> 2
- net /I2C_GP0_DAT_1V8_J: track 28.7 -> 62.4 mm, vias 0 -> 2
- net /CAM0_RST: track 0.00 -> 33.6 mm, vias 0 -> 1
- net /CAM0_RST_J: track 30.9 -> 64.1 mm, vias 0 -> 1
- net /CAM_I2C2_SDA_J: track 26.5 -> 59.1 mm, vias 0 -> 2
- net /CAM2_MCLK: track 0.00 -> 32.5 mm
- net /I2S3_SDIN: track 0.00 -> 32.4 mm, vias 0 -> 2
- net /CAM2_RST: track 0.00 -> 31.6 mm, vias 0 -> 1
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Other:
- net class Default: trace_width 0.3048 -> 0.2032

Commit message: DRC OK
Routing:
- net /AVDD_CAM: track 0.00 -> 45.7 mm, vias 0 -> 2
- net /CAM_VSYNC: track 0.00 -> 28.3 mm, vias 0 -> 3
- net /VDD_AF: track 0.00 -> 27.7 mm, vias 0 -> 3
- net /CAM_AF_PWDN: track 0.00 -> 27.4 mm, vias 0 -> 2
- net /I2C_CAM_DAT: track 25.9 -> 27.5 mm
- net /CAM_I2C2_SCL_J: track 60.2 -> 61.8 mm
- net Earth: vias 245 -> 244
Other:
- net class Default: clearance 0.1778 -> 0.1524
- rule trace_clearance: 0.1778 -> 0.1524
