File: Jetson_camera_interposer.sch (KiCad schematic (older format))
At the start: 21 parts, among them J1 QSH-060-01-L-D-A, J2 QTH-060-01-L-D-A, J21 Conn_01x01, J22 Conn_01x01, J23 Conn_01x01, J24 Conn_01x01, J25 Conn_01x01, J26 Conn_01x01, J3 Conn_01x01, J4 Conn_01x01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

Commit message: finished routing second connector
Connections:
- net labels added: CAM0_MCLK_J, CAM0_RST_J, CAM1_MCLK_J, CAM1_RST_L_J, CAM2_MCLK_J, CAM2_RST_J, CAM_I2C2_SCL_J, CAM_I2C2_SDA_J, I2C_CAM_CLK_J, I2C_CAM_DAT_J, I2C_GP0_CLK_1V8_J, I2C_GP0_DAT_1V8_J
- wire segments 343 -> 355
Changed lines of the file:
@@
 CAM0_PWR
 Text Label 1500 6600 2    60   ~ 0
-CAM0_RST
+CAM0_RST_J
 Text Label 1500 6700 2    60   ~ 0
 CAM_FLASH_EN
@@
 NoConn ~ 8100 5500
 Text Label 7400 5600 2    60   ~ 0
-I2C_CAM_CLK
+I2C_CAM_CLK_J
 Text Label 7450 5750 2    60   ~ 0
-I2C_CAM_DAT
+I2C_CAM_DAT_J
 Text Label 7350 6400 2    60   ~ 0
-CAM0_MCLK
+CAM0_MCLK_J
 Text Label 7300 6500 2    60   ~ 0
 CAM0_PWR
 Text Label 7250 6600 2    60   ~ 0
-CAM0_RST
+CAM0_RST_J
 Text Label 7450 6700 2    60   ~ 0
 CAM_FLASH_EN
@@
 JETSON_1V2_J
 Text Label 7500 7100 2    60   ~ 0
-I2C_GP0_CLK_1V8
+I2C_GP0_CLK_1V8_J
 Text Label 7300 7200 2    60   ~ 0
-I2C_GP0_DAT_1V8
+I2C_GP0_DAT_1V8_J
 Text Label 10750 6100 0    60   ~ 0
 CAM_VSYNC
@@
 	9750 6700 10350 6700
 Text Label 10350 6200 0    60   ~ 0
-CAM1_MCLK
+CAM1_MCLK_J
 Text Label 10350 6300 0    60   ~ 0
 CAM1_PWDN
 Text Label 10350 6400 0    60   ~ 0
-CAM1_RST_L
+CAM1_RST_L_J
 Text Label 10350 6500 0    60   ~ 0
-CAM2_MCLK
+CAM2_MCLK_J
 Text Label 10350 6600 0    60   ~ 0
 CAM2_PWDN
 Text Label 10350 6700 0    60   ~ 0
-CAM2_RST
+CAM2_RST_J
 $Comp
 L TX2_Symbols:QTH-060-01-L-D-A J2
@@
 	8100 6300 6950 6300
 Text Label 6950 6200 0    60   ~ 0
-CAM_I2C2_SCL
+CAM_I2C2_SCL_J
 Text Label 6950 6300 0    60   ~ 0
-CAM_I2C2_SDA
+CAM_I2C2_SDA_J
 Wire Wire Line
 	2500 6200 950  6200
@@
 Text Label 14700 4200 2    60   ~ 0
 CAM0_MCLK
-Text Label 14850 6100 2    60   ~ 0
+Text Label 14700 6450 2    60   ~ 0
 CAM0_PWR
 Text Label 15650 1600 2    60   ~ 0
@@
 Text Label 14200 4000 0    60   ~ 0
 CAM1_MCLK
-Text Label 14400 6200 0    60   ~ 0
-CAM1_PWDN
 Text Label 14200 3800 0    60   ~ 0
 CAM2_MCLK
-Text Label 14400 6300 0    60   ~ 0
-CAM2_PWDN
 Text Label 14250 3700 0    60   ~ 0
 CAM2_RST
@@
 Wire Wire Line
 	14050 4200 14700 4200
+Text Label 12750 3700 0    60   ~ 0
+CAM2_RST_J
+Text Label 12650 3800 0    60   ~ 0
+CAM2_MCLK_J
+Text Label 12650 3900 0    60   ~ 0
+CAM1_RST_L_J
+Text Label 12650 4000 0    60   ~ 0
+CAM1_MCLK_J
+Text Label 13250 4100 2    60   ~ 0
+CAM0_RST_J
+Text Label 13250 4200 2    60   ~ 0
+CAM0_MCLK_J
+Text Label 13250 4300 2    60   ~ 0
+I2C_GP0_DAT_1V8_J
+Text Label 13250 4400 2    60   ~ 0
+I2C_GP0_CLK_1V8_J
+Text Label 12500 4500 0    60   ~ 0
+CAM_I2C2_SDA_J
+Text Label 12500 4600 0    60   ~ 0
+CAM_I2C2_SCL_J
+Text Label 13250 4700 2    60   ~ 0
+I2C_CAM_DAT_J
+Text Label 13250 4800 2    60   ~ 0
+I2C_CAM_CLK_J
+Wire Wire Line
+	13550 3700 12750 3700
+Wire Wire Line
+	13550 3800 12650 3800
+Wire Wire Line
+	13550 3900 12650 3900
+Wire Wire Line
+	13550 4000 12650 4000
+Wire Wire Line
+	13550 4100 13250 4100
+Wire Wire Line
+	13250 4200 13550 4200
+Wire Wire Line
+	13550 4300 13250 4300
+Wire Wire Line
+	13550 4400 13250 4400
+Wire Wire Line
+	13550 4500 12500 4500
+Wire Wire Line
+	13550 4600 12500 4600
+Wire Wire Line
+	13550 4700 13250 4700
+Wire Wire Line
+	13250 4800 13550 4800
+Text Label 14250 6650 0    60   ~ 0
+CAM2_PWDN
+Text Label 14250 6550 0    60   ~ 0
+CAM1_PWDN
 $EndSCHEMATC

Commit message: finished third connector
Connections:
- net labels added: CAM0_PWR_J, CAM1_PWDN_J, CAM2_PWDN_J, CAM_INTR_J, CAM_VSYNC_J, VSYS_EN_J
- wire segments 355 -> 367
Changed lines of the file:
@@
 Text Label 1500 6700 2    60   ~ 0
 CAM_FLASH_EN
-Text Label 4850 6100 2    60   ~ 0
-CAM_VSYNC
 $Comp
 L power:Earth #PWR01
@@
 CAM0_MCLK_J
 Text Label 7300 6500 2    60   ~ 0
-CAM0_PWR
+CAM0_PWR_J
 Text Label 7250 6600 2    60   ~ 0
 CAM0_RST_J
@@
 I2C_GP0_DAT_1V8_J
 Text Label 10750 6100 0    60   ~ 0
-CAM_VSYNC
+CAM_VSYNC_J
 Text Label 11200 6900 0    60   ~ 0
 JETSON_1V8_J
@@
 IR_TRIGGER
 Text Label 7200 7700 0    60   ~ 0
-CAM_INTR
+CAM_INTR_J
 Text Label 7250 7800 0    60   ~ 0
-VSYS_EN
+VSYS_EN_J
 Text Label 2250 7300 2    60   ~ 0
 VDD_IR
@@
 CAM1_MCLK_J
 Text Label 10350 6300 0    60   ~ 0
-CAM1_PWDN
+CAM1_PWDN_J
 Text Label 10350 6400 0    60   ~ 0
 CAM1_RST_L_J
@@
 CAM2_MCLK_J
 Text Label 10350 6600 0    60   ~ 0
-CAM2_PWDN
+CAM2_PWDN_J
 Text Label 10350 6700 0    60   ~ 0
 CAM2_RST_J
@@
 Text Label 14700 4200 2    60   ~ 0
 CAM0_MCLK
-Text Label 14700 6450 2    60   ~ 0
+Text Label 14650 6400 2    60   ~ 0
 CAM0_PWR
 Text Label 15650 1600 2    60   ~ 0
@@
 Text Label 15050 1800 0    60   ~ 0
 IR_TRIGGER
-Text Label 15050 1950 0    60   ~ 0
+Text Label 14200 6700 0    60   ~ 0
 CAM_INTR
-Text Label 15050 2100 0    60   ~ 0
+Text Label 14200 6800 0    60   ~ 0
 VSYS_EN
 Text Label 15050 2750 0    60   ~ 0
@@
 Text Label 15100 3100 0    60   ~ 0
 I2S3_SDOUT
-Text Label 15050 2250 0    60   ~ 0
+Text Label 14200 6900 0    60   ~ 0
 CAM_VSYNC
 Text Label 14200 4000 0    60   ~ 0
@@
 U 1 1 61A4E08F
 P 13800 6600
-F 0 "J9" H 13850 7317 50  0000 C CNN
-F 1 "Conn_02x30_Odd_Even" H 13850 7226 50  0000 C CNN
+F 0 "J9" H 13850 7050 50  0000 C CNN
+F 1 "Conn_02x30_Odd_Even" H 13850 6950 50  0000 C CNN
 F 2 "Pin_Headers:Pin_Header_Straight_2x06_Pitch2.54mm" H 13800 6600 50  0001 C CNN
 F 3 "~" H 13800 6600 50  0001 C CNN
@@
 Wire Wire Line
 	13250 4800 13550 4800
-Text Label 14250 6650 0    60   ~ 0
+Text Label 14200 6600 0    60   ~ 0
 CAM2_PWDN
-Text Label 14250 6550 0    60   ~ 0
+Text Label 14200 6500 0    60   ~ 0
 CAM1_PWDN
+Wire Wire Line
+	14100 6400 14650 6400
+Wire Wire Line
+	14100 6500 14200 6500
+Wire Wire Line
+	14100 6600 14200 6600
+Wire Wire Line
+	14100 6700 14200 6700
+Wire Wire Line
+	14100 6800 14200 6800
+Wire Wire Line
+	14100 6900 14200 6900
+Text Label 13300 6400 2    60   ~ 0
+CAM0_PWR_J
+Text Label 12800 6500 0    60   ~ 0
+CAM1_PWDN_J
+Text Label 12800 6600 0    60   ~ 0
+CAM2_PWDN_J
+Text Label 12900 6700 0    60   ~ 0
+CAM_INTR_J
+Text Label 12950 6800 0    60   ~ 0
+VSYS_EN_J
+Text Label 12850 6900 0    60   ~ 0
+CAM_VSYNC_J
+Wire Wire Line
+	13300 6400 13600 6400
+Wire Wire Line
+	12800 6500 13600 6500
+Wire Wire Line
+	12800 6600 13600 6600
+Wire Wire Line
+	12900 6700 13600 6700
+Wire Wire Line
+	12950 6800 13600 6800
+Text Label 4850 6100 2    60   ~ 0
+CAM_VSYNC
+Wire Wire Line
+	12850 6900 13600 6900
 $EndSCHEMATC

Commit message: before re-arranging connectors
Other:
- note added: "VERY BAD LOCATION, FMC DOESN'T FIT. MOVE IT!!!"
Changed lines of the file:
@@
 Wire Wire Line
 	12850 6900 13600 6900
+Text Notes 12450 3450 0    60   Italic 12
+VERY BAD LOCATION, FMC DOESN'T FIT. MOVE IT!!!
 $EndSCHEMATC

Commit message: reset all wirings
Parts:
- removed J7: Conn_02x10_Odd_Even, Pin_Headers:Pin_Header_Straight_2x10_Pitch2.54mm, symbol Connector_Generic:Conn_02x10_Odd_Even
- removed J9: Conn_02x30_Odd_Even, Pin_Headers:Pin_Header_Straight_2x06_Pitch2.54mm, symbol Connector_Generic:Conn_02x06_Odd_Even
Connections:
- wire segments 367 -> 348
Changed lines of the file:
@@
 Text Label 4750 5700 0    60   ~ 0
 I2S3_SDOUT
-$Comp
-L Connector_Generic:Conn_02x10_Odd_Even J7
-U 1 1 615E8738
-P 13050 8300
-F 0 "J7" H 13100 8917 50  0000 C CNN
-F 1 "Conn_02x10_Odd_Even" H 13100 8826 50  0000 C CNN
-F 2 "Pin_Headers:Pin_Header_Straight_2x10_Pitch2.54mm" H 13050 8300 50  0001 C CNN
-F 3 "~" H 13050 8300 50  0001 C CNN
-	1    13050 8300
-	1    0    0    -1
-$EndComp
-Wire Wire Line
-	12850 8100 11850 8100
-Wire Wire Line
-	12850 8200 11850 8200
-Wire Wire Line
-	12850 8300 11850 8300
-Wire Wire Line
-	12850 8400 11850 8400
-Wire Wire Line
-	12850 8500 11850 8500
-Wire Wire Line
-	12850 8600 11850 8600
-Wire Wire Line
-	12850 8700 11850 8700
-Wire Wire Line
-	12850 8800 12350 8800
-Wire Wire Line
-	13350 8800 13850 8800
-Wire Wire Line
-	13350 8700 13850 8700
-Wire Wire Line
-	13350 8600 13850 8600
-Wire Wire Line
-	13350 8500 13850 8500
-Wire Wire Line
-	13350 8400 13850 8400
-Wire Wire Line
-	13350 8300 13850 8300
-Wire Wire Line
-	13350 8200 13850 8200
-Wire Wire Line
-	13350 8100 13850 8100
 Text Label 13850 7900 0    60   ~ 0
 VDD_SYS_J
@@
 Text Label 11850 8700 0    60   ~ 0
 DVDD_CAM_LV
-$Comp
-L power:Earth #PWR0101
-U 1 1 61B5BBC6
-P 12350 8950
-F 0 "#PWR0101" H 12350 8700 50  0001 C CNN
-F 1 "Earth" H 12350 8800 50  0001 C CNN
-F 2 "" H 12350 8950 50  0000 C CNN
-F 3 "" H 12350 8950 50  0000 C CNN
-	1    12350 8950
-	1    0    0    -1
-$EndComp
-Wire Wire Line
-	12350 8800 12350 8950
-$Comp
-L power:Earth #PWR0102
-U 1 1 61B84369
-P 13850 8950
-F 0 "#PWR0102" H 13850 8700 50  0001 C CNN
-F 1 "Earth" H 13850 8800 50  0001 C CNN
-F 2 "" H 13850 8950 50  0000 C CNN
-F 3 "" H 13850 8950 50  0000 C CNN
-	1    13850 8950
-	1    0    0    -1
-$EndComp
-Wire Wire Line
-	13850 8800 13850 8950
 Text Label 11850 7900 0    60   ~ 0
 VDD_SYS
@@
 Text Label 14700 4200 2    60   ~ 0
 CAM0_MCLK
-Text Label 14650 6400 2    60   ~ 0
-CAM0_PWR
 Text Label 15650 1600 2    60   ~ 0
 CAM_FLASH_EN
@@
 Text Label 15050 1800 0    60   ~ 0
 IR_TRIGGER
-Text Label 14200 6700 0    60   ~ 0
-CAM_INTR
-Text Label 14200 6800 0    60   ~ 0
-VSYS_EN
 Text Label 15050 2750 0    60   ~ 0
 I2S3_CLK
@@
 Text Label 15100 3100 0    60   ~ 0
 I2S3_SDOUT
-Text Label 14200 6900 0    60   ~ 0
-CAM_VSYNC
 Text Label 14200 4000 0    60   ~ 0
 CAM1_MCLK
@@
 	1    0    0    -1
 $EndComp
-Wire Wire Line
-	12850 7900 11850 7900
-Wire Wire Line
-	12850 8000 11850 8000
-Wire Wire Line
-	13350 7900 13850 7900
-Wire Wire Line
-	13350 8000 13850 8000
 Text Label 14200 3900 0    60   ~ 0
 CAM1_RST_L
-$Comp
-L Connector_Generic:Conn_02x06_Odd_Even J9
-U 1 1 61A4E08F
-P 13800 6600
-F 0 "J9" H 13850 7050 50  0000 C CNN
-F 1 "Conn_02x30_Odd_Even" H 13850 6950 50  0000 C CNN
-F 2 "Pin_Headers:Pin_Header_Straight_2x06_Pitch2.54mm" H 13800 6600 50  0001 C CNN
-F 3 "~" H 13800 6600 50  0001 C CNN
-	1    13800 6600
-	1    0    0    -1
-$EndComp
 Text Label 14950 4300 2    60   ~ 0
 I2C_GP0_DAT_1V8
@@
 Wire Wire Line
 	13250 4800 13550 4800
+Text Label 4850 6100 2    60   ~ 0
+CAM_VSYNC
+Text Notes 12450 3450 0    60   Italic 12
+VERY BAD LOCATION, FMC DOESN'T FIT. MOVE IT!!!
+Text Label 12850 6900 0    60   ~ 0
+CAM_VSYNC_J
+Text Label 12950 6800 0    60   ~ 0
+VSYS_EN_J
+Text Label 12900 6700 0    60   ~ 0
+CAM_INTR_J
+Text Label 12800 6600 0    60   ~ 0
+CAM2_PWDN_J
+Text Label 12800 6500 0    60   ~ 0
+CAM1_PWDN_J
+Text Label 13300 6400 2    60   ~ 0
+CAM0_PWR_J
+Text Label 14200 6500 0    60   ~ 0
+CAM1_PWDN
 Text Label 14200 6600 0    60   ~ 0
 CAM2_PWDN
-Text Label 14200 6500 0    60   ~ 0
-CAM1_PWDN
-Wire Wire Line
-	14100 6400 14650 6400
-Wire Wire Line
-	14100 6500 14200 6500
-Wire Wire Line
-	14100 6600 14200 6600
-Wire Wire Line
-	14100 6700 14200 6700
-Wire Wire Line
-	14100 6800 14200 6800
-Wire Wire Line
-	14100 6900 14200 6900
-Text Label 13300 6400 2    60   ~ 0
-CAM0_PWR_J
-Text Label 12800 6500 0    60   ~ 0
-CAM1_PWDN_J
-Text Label 12800 6600 0    60   ~ 0
-CAM2_PWDN_J
-Text Label 12900 6700 0    60   ~ 0
-CAM_INTR_J
-Text Label 12950 6800 0    60   ~ 0
-VSYS_EN_J
-Text Label 12850 6900 0    60   ~ 0
-CAM_VSYNC_J
-Wire Wire Line
-	13300 6400 13600 6400
-Wire Wire Line
-	12800 6500 13600 6500
-Wire Wire Line
-	12800 6600 13600 6600
-Wire Wire Line
-	12900 6700 13600 6700
-Wire Wire Line
-	12950 6800 13600 6800
-Text Label 4850 6100 2    60   ~ 0
+Text Label 14200 6900 0    60   ~ 0
 CAM_VSYNC
-Wire Wire Line
-	12850 6900 13600 6900
-Text Notes 12450 3450 0    60   Italic 12
-VERY BAD LOCATION, FMC DOESN'T FIT. MOVE IT!!!
+Text Label 14200 6800 0    60   ~ 0
+VSYS_EN
+Text Label 14200 6700 0    60   ~ 0
+CAM_INTR
+Text Label 14650 6400 2    60   ~ 0
+CAM0_PWR
+Wire Wire Line
+	11850 7900 13850 7900
+Wire Wire Line
+	11850 8000 13850 8000
+Wire Wire Line
+	11850 8100 13850 8100
+Wire Wire Line
+	11850 8200 13850 8200
+Wire Wire Line
+	11850 8300 13850 8300
+Wire Wire Line
+	11850 8400 13850 8400
+Wire Wire Line
+	11850 8500 13850 8500
+Wire Wire Line
+	11850 8600 13850 8600
+Wire Wire Line
+	11850 8700 13850 8700
+Wire Wire Line
+	13300 6400 14650 6400
+Wire Wire Line
+	12800 6500 14200 6500
+Wire Wire Line
+	12800 6600 14200 6600
+Wire Wire Line
+	12900 6700 14200 6700
+Wire Wire Line
+	12950 6800 14200 6800
+Wire Wire Line
+	12850 6900 14200 6900
 $EndSCHEMATC
